File: V1/ESC_V1.kicad_pcb (KiCad board)
At the start: 2 copper layers, 53 parts, among them J1 USB_C_Receptacle_USB2.0, Q1 Q_NMOS_GDS, Q2 Q_NMOS_GDS, Q3 Q_NMOS_GDS, Q4 Q_NMOS_GDS, Q5 Q_NMOS_GDS, Q6 Q_NMOS_GDS, U1 IRS2001, U2 ATmega328P-AU_full, U3 IRS2001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

Commit message: aaa
Parts:
- C10, R10, R11, R13, R14, R16, R17, R18, R8, R9: moved to B.Cu
- J1: footprint Connector_USB:USB_C_Receptacle_GCT_USB4105-xx-A_16P_TopMnt_Horizontal -> Dam_libkicad:USB-C USB4110_GCT
- moved D5 113.4 mm to (130.4, 110.0), turned to 90 degrees
- moved F1 112.5 mm to (126.5, 109.4), turned to 180 degrees
- moved D6 109.5 mm to (132.8, 110.0), turned to 90 degrees
- moved R14 97.6 mm to (138.4, 111.1), turned to 180 degrees
- moved U3 96.6 mm to (154.6, 93.7), turned to 90 degrees
- moved U4 96.1 mm to (137.7, 93.7), turned to 90 degrees
- moved R15 95.9 mm to (132.8, 105.4), turned to -90 degrees
- moved R16 95.4 mm to (145.2, 120.3)
- moved C4 94.4 mm to (148.5, 97.5), turned to -90 degrees
- moved C5 94.1 mm to (131.6, 97.5), turned to -90 degrees
- moved U6 93.9 mm to (166.2, 60.6)
- moved C3 93.9 mm to (163.7, 99.1)
- moved D1 93.9 mm to (168.4, 99.1)
- moved Q2 93.9 mm to (167.6, 72.7)
- moved Q3 93.9 mm to (151.2, 76.4)
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Connections:
- C6 pad 2: D+ -> Net-(U5-3V3OUT)
- J1 pad A7: D+ -> D-
- J1 pad B7: D+ -> D-
- U5 pad 10: D+ -> Net-(U5-3V3OUT)
- U5 pad 11: D+ -> unconnected-(U5-~{RESET}-Pad11)
- U5 pad 3: D+ -> Net-(U5-3V3OUT)
- U5 pad 9: D+ -> D-
Routing:
- net GND: track 127.3 -> 250.7 mm, vias 3 -> 9
- net MOTOR_V: track 29.7 -> 111.6 mm, vias 0 -> 1
- net MOTOR_U: track 29.9 -> 109.9 mm, vias 0 -> 1
- net MOTOR_W: track 32.6 -> 103.2 mm, vias 0 -> 1
- net +5V: track 12.7 -> 60.7 mm
- net RXu_0: track 0.00 -> 36.1 mm, vias 0 -> 2
- net PHV_U: track 0.00 -> 34.3 mm, vias 0 -> 1
- net TXu_0: track 0.00 -> 33.1 mm, vias 0 -> 2
- net PHV_V: track 0.00 -> 28.3 mm, vias 0 -> 1
- net PHV_W: track 0.00 -> 24.4 mm, vias 0 -> 1
- net Net-(U5-3V3OUT): track 0.00 -> 22.2 mm
- net V_BAT: track 146.1 -> 125.4 mm
- net RST: track 0.00 -> 20.5 mm
- net Net-(F1-Pad2): track 0.00 -> 17.0 mm
- net PWM_A_L: track 35.7 -> 19.0 mm
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- added copper zone on B.Cu, net GND
- added copper zone on F.Cu, net GND
Other:
- board outline added: 55.9 x 68.3 mm

Commit message: aaa
Parts:
- added C11: 1uF, Dam_libkicad:0603, F.Cu at (144.3, 109.5)
- added C12: 1uF, Dam_libkicad:0603, F.Cu at (140.9, 105.2)
- added C13: 10uF, Dam_libkicad:0603, F.Cu at (167.3, 99.3)
- added C14: 10uF, Dam_libkicad:0603, F.Cu at (148.8, 98.1)
- added C15: 10uF, Dam_libkicad:0603, F.Cu at (132.2, 99.8)
- added J3: Conn_01x03, Connector_PinSocket_2.54mm:PinSocket_1x03_P2.54mm_Horizontal, F.Cu at (164.9, 123.3)
- added JP1: Jumper_2_Open, TestPoint:TestPoint_2Pads_Pitch2.54mm_Drill0.8mm, F.Cu at (136.2, 103.5)
- added R19: 10k, Dam_libkicad:1206, F.Cu at (145.8, 110.1)
- added U12: MIC5205-5.0YM5, Package_TO_SOT_SMD:TSOT-23-5, F.Cu at (143.3, 105.9)
- C1, C2: footprint Dam_libkicad:1206 -> Dam_libkicad:0603
- C3, C4, C5: value C -> 2.2uF; footprint Dam_libkicad:1206 -> Dam_libkicad:0603
- D1, D2, D3: value D -> 1N4148WS
- D5, D6: footprint LED_SMD:LED_1206_3216Metric_Pad1.42x1.75mm_HandSolder -> LED_SMD:LED_0603_1608Metric
- R10, R11, R13, R14, R8, R9: value R -> 33k
- R16, R17, R18: value R -> 10k
- moved R1 8.88 mm to (161.0, 85.8)
- moved Y1 7.15 mm to (168.0, 105.8), turned to 0 degrees
- moved C10 6.51 mm to (159.6, 110.0)
- moved U2 5.72 mm to (159.9, 110.2)
- moved C2 5.50 mm to (151.5, 109.4)
- moved C1 5.39 mm to (152.6, 109.4)
- moved R2 4.70 mm to (165.0, 85.8)
- moved C3 3.84 mm to (164.1, 95.2), turned to -90 degrees
- moved D1 3.76 mm to (166.2, 96.0), turned to -90 degrees
- moved R17 3.40 mm to (145.2, 114.9)
- moved R18 3.40 mm to (145.2, 112.9)
- moved R16 3.30 mm to (145.2, 117.0)
- moved R5 2.77 mm to (127.5, 85.5)
- moved U1 2.63 mm to (170.1, 95.0), turned to 90 degrees
- moved U10 2.35 mm to (122.5, 85.8)
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Connections:
- U1 pad 4: unconnected-(U1-COM-Pad4) -> GND
- U2 pad 20: unconnected-(U2-AREF-Pad20) -> Net-(U2-AREF)
- U2 pad 32: unconnected-(U2-(2/INT0)PD2-Pad32) -> PWM_IN
- U3 pad 4: unconnected-(U3-COM-Pad4) -> GND
- U4 pad 4: unconnected-(U4-COM-Pad4) -> GND
Routing:
- net GND: track 250.7 -> 398.1 mm, vias 9 -> 23
- net +5V: track 60.7 -> 97.2 mm, vias 0 -> 1
- net RST: track 20.5 -> 33.9 mm
- net PWM_IN: track 0.00 -> 11.8 mm, vias 0 -> 1
- net Net-(JP1-B): track 0.00 -> 10.7 mm
- net Net-(U1-LO): track 1.46 -> 11.2 mm
- net Net-(U1-HO): track 3.39 -> 12.6 mm
- net Net-(Q1-G): track 28.4 -> 19.2 mm
- net V_BAT: track 125.4 -> 132.4 mm
- net MOTOR_V: track 111.6 -> 104.8 mm
- net PWM_B_L: track 18.6 -> 12.2 mm
- net MOTOR_U: track 109.9 -> 116.0 mm
- net PWM_B_H: track 17.4 -> 11.7 mm
- net PHV_W: track 24.4 -> 19.1 mm
- net MOTOR_W: track 103.2 -> 98.0 mm
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- removed copper zone on B.Cu, net GND
- removed copper zone on F.Cu, net GND

Commit message: v2 80%
Parts:
- removed F1: Fuse, Fuse:Fuse_1206_3216Metric_Pad1.42x1.75mm_HandSolder
- C13, C14, C15, C3, C4, C5: footprint Dam_libkicad:0603 -> Dam_libkicad:1206
- moved R9 17.7 mm to (155.0, 100.8), turned to 90 degrees
- moved R14 10.4 mm to (139.7, 100.8), turned to 90 degrees
- moved R11 9.24 mm to (142.7, 100.8), turned to 90 degrees
- moved C4 7.72 mm to (144.2, 89.3), turned to 180 degrees
- moved C10 5.53 mm to (164.3, 107.0)
- moved D2 3.83 mm to (150.9, 93.7)
- moved D3 3.49 mm to (133.5, 94.0)
- moved Y1 3.18 mm to (168.4, 109.0), turned to 180 degrees
- moved U9 2.78 mm to (122.2, 75.1)
- moved C13 2.63 mm to (164.7, 99.2)
- moved C5 2.16 mm to (131.2, 93.3), turned to -90 degrees
- moved C15 2.02 mm to (133.6, 98.3)
- moved R1 1.95 mm to (162.9, 85.8)
- moved R5 1.86 mm to (129.3, 85.7)
- moved C14 1.53 mm to (148.9, 96.5), turned to -90 degrees
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Connections:
- J1 pad A4: Net-(F1-Pad2) -> +5V
- J1 pad A9: Net-(F1-Pad2) -> +5V
- U2 pad 1: PWM_A_L -> PWM_B_L
- U2 pad 10: PWM_B_L -> VIRTUAL_N
- U2 pad 11: VIRTUAL_N -> unconnected-(U2-(7/AIN1)PD7-Pad11)
- U2 pad 12: unconnected-(U2-(8)PB0-Pad12) -> PWM_IN
- U2 pad 13: PWM_B_H -> PWM_A_H
- U2 pad 14: PWM_C_L -> PWM_B_H
- U2 pad 2: unconnected-(U2-(4/T0)PD4-Pad2) -> PWM_A_L
- U2 pad 20: Net-(U2-AREF) -> unconnected-(U2-AREF-Pad20)
- U2 pad 32: PWM_IN -> PWM_C_L
- U2 pad 9: PWM_A_H -> unconnected-(U2-(5/OC0B/T1)PD5-Pad9)
Routing:
- net PWM_C_L: track 25.9 -> 60.9 mm, vias 0 -> 2
- net MOTOR_U: track 116.0 -> 85.5 mm
- net PWM_B_L: track 12.2 -> 37.9 mm, vias 0 -> 2
- net PWM_IN: track 11.8 -> 36.2 mm, vias 1 -> 2
- net MOTOR_V: track 104.8 -> 80.9 mm
- net +5V: track 97.2 -> 117.7 mm
- net Net-(F1-Pad2): track 17.0 -> 0.00 mm
- net VIRTUAL_N: track 16.9 -> 25.7 mm
- net PHV_W: track 19.1 -> 26.6 mm
- net Net-(D3-K): track 13.2 -> 6.37 mm, vias 2 -> 0
- net MOTOR_W: track 98.0 -> 91.3 mm
- net PWM_A_H: track 11.9 -> 17.4 mm
- net V_BAT: track 132.4 -> 136.8 mm
- net Net-(D2-K): track 12.9 -> 9.03 mm, vias 2 -> 0
- net GND: track 398.1 -> 394.5 mm, vias 23 -> 21
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