File: V1/ESC_V1.kicad_sch (KiCad schematic)
At the start: 53 parts, among them J1 USB_C_Receptacle_USB2.0, Q1 Q_NMOS_GDS, Q2 Q_NMOS_GDS, Q3 Q_NMOS_GDS, Q4 Q_NMOS_GDS, Q5 Q_NMOS_GDS, Q6 Q_NMOS_GDS, U1 IRS2001, U2 ATmega328P-AU_full, U3 IRS2001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

Commit message: aaa
Parts:
- J1: footprint Dam_libkicad:USB4125 -> Dam_libkicad:USB-C USB4110_GCT

Commit message: aaa
Parts:
- added C11, C12: 1uF, Dam_libkicad:0603, symbol Device:C
- added C13, C14, C15: 10uF, Dam_libkicad:0603, symbol Device:C
- added J3: Conn_01x03, Connector_PinSocket_2.54mm:PinSocket_1x03_P2.54mm_Horizontal, symbol Connector_Generic:Conn_01x03
- added JP1: Jumper_2_Open, TestPoint:TestPoint_2Pads_Pitch2.54mm_Drill0.8mm, symbol Jumper:Jumper_2_Open
- added R19: 10k, Dam_libkicad:1206, symbol Device:R
- added U12: MIC5205-5.0YM5, Package_TO_SOT_SMD:TSOT-23-5, symbol Regulator_Linear:MIC5205-5.0YM5
- C1, C2: footprint Dam_libkicad:1206 -> Dam_libkicad:0603
- C3, C4, C5: value C -> 2.2uF; footprint Dam_libkicad:1206 -> Dam_libkicad:0603
- D1, D2, D3: value D -> 1N4148WS
- D5, D6: footprint LED_SMD:LED_1206_3216Metric_Pad1.42x1.75mm_HandSolder -> LED_SMD:LED_0603_1608Metric
- R10, R11, R13, R14, R8, R9: value R -> 33k
- R16, R17, R18: value R -> 10k
Connections:
- net +5V: now also C11.1, J3.1 (Pin_1), R19.2, U12.5 (OUT)
- net GND: now also U1.4 (COM), U3.4 (COM), U4.4 (COM), C11.2, C12.2, C13.2, C14.2, C15.2, J3.3 (Pin_3), U12.2 (GND)
- net RST: now also R19.1
- net V_BAT: now also C13.1, C14.1, C15.1, JP1.1 (A)
- net PWM_IN: now reaches U2.32 ((2/INT0)PD2)
- net PWM_IN: now also J3.2 (Pin_2)
- new net: C12.1, JP1.2 (B), U12.1 (IN), U12.3 (EN)
- no-connect marks 0 -> 1
Other:
- moved on the sheet: C1, C2, D5, D6, U10, U2, U5, U9, Y1

Commit message: v2 80%
Parts:
- removed F1: Fuse, Fuse:Fuse_1206_3216Metric_Pad1.42x1.75mm_HandSolder, symbol Device:Fuse
- C13, C14, C15, C3, C4, C5: footprint Dam_libkicad:0603 -> Dam_libkicad:1206
Connections:
- net +5V: now also J1.A4 (VBUS), J1.A9 (VBUS), J1.B4 (VBUS), J1.B9 (VBUS)
- net PWM_A_H: now also U2.13 ((9/OC1A)PB1); no longer U2.9 ((5/OC0B/T1)PD5)
- net PWM_A_L: now also U2.2 ((4/T0)PD4); no longer U2.1 ((3/OC2B/INT1)PD3)
- net PWM_B_H: now also U2.14 ((10/OC1B/~{SS})PB2); no longer U2.13 ((9/OC1A)PB1)
- net PWM_B_L: now also U2.1 ((3/OC2B/INT1)PD3); no longer U2.10 ((6/OC0A/AIN0)PD6)
- net PWM_C_L: now also U2.32 ((2/INT0)PD2); no longer U2.14 ((10/OC1B/~{SS})PB2)
- net PWM_IN: now also U2.12 ((8)PB0); no longer U2.32 ((2/INT0)PD2)
- net VIRTUAL_N: now also U2.10 ((6/OC0A/AIN0)PD6); no longer U2.11 ((7/AIN1)PD7)
