File: V2/ESC.kicad_pcb (KiCad board)
At the start: 2 copper layers, 126 parts, among them IC1 DRV8302DCA, IC2 TPS54331DR, J1 Conn_01x01, J2 Conn_01x01, J3 Conn_01x01, J4 Prog, J6 USB_C_Receptacle_USB2.0, Q1 2N7002, Q2 NMOS, Q3 NMOS, Q4 NMOS, Q5 NMOS, Q6 NMOS, Q7 NMOS, U1 ATmega328P-AU_full, U2 FT230XS, U5 LMV321, U6 LMV321, U7 LMV321, Y1 CSTCE

Commit message: def
Parts:
- removed 6.8uH/4A1: L2, Inductor_SMD:L_1206_3216Metric
- removed C10: 0.1uF, Capacitor_SMD:C_1206_3216Metric
- removed C11, C29, C32: 4.7uF, Capacitor_SMD:C_1206_3216Metric
- removed C12, C13, C14, C15: C_Polarized, Capacitor_SMD:CP_Elec_4x3
- removed C16, C17, C18, C19, C20, C21, C22: C, Capacitor_SMD:C_0201_0603Metric
- removed C30, C31: 10nF, Capacitor_SMD:C_1206_3216Metric
- removed C33: 2.2nF, Capacitor_SMD:C_1206_3216Metric
- removed C34, C41: 47uF, Capacitor_SMD:C_1206_3216Metric
- removed C35, C36, C37, C38, C39, C40: 1nF, Capacitor_SMD:C_1206_3216Metric
- removed C42: 1000pF, Capacitor_SMD:C_1206_3216Metric
- removed C43: 47pF, Capacitor_SMD:C_1206_3216Metric
- removed C8: C, Capacitor_SMD:C_1206_3216Metric
- removed D1, D2, D3: ZMMxx, Diode_SMD:D_MiniMELF
- removed D4: ESD131-B1-W0201, Diode_SMD:Infineon_SG-WLL-2-3_0.58x0.28_P0.36mm
- removed D6: BAT85, Diode_THT:D_DO-35_SOD27_P7.62mm_Horizontal
- removed IC2: TPS54331DR, Dam_libkicad:SOIC127P600X175-8N
- removed J1, J2, J3: Conn_01x01, Connector_JST:JST_ACH_BM01B-ACHSS-A-GAN-ETF_1x01-1MP_P1.20mm_Vertical
- removed J4: Prog, Connector_PinHeader_2.54mm:PinHeader_1x04_P2.54mm_Vertical
- removed L1: L, Inductor_SMD:L_1206_3216Metric
- removed Q1: 2N7002, Package_TO_SOT_SMD:SOT-23
- removed R10, R37, R44: 10k, Resistor_SMD:R_1206_3216Metric
- removed R11, R12, R13, R14, R15, R16, R17, R18, R19, R20, R21, R22: 10, Resistor_SMD:R_1206_3216Metric
- removed R23, R39, R40, R41: R, Resistor_SMD:R_1206_3216Metric
- removed R36: 15k, Resistor_SMD:R_1206_3216Metric
- removed R38: 2.2k, Resistor_SMD:R_1206_3216Metric
- removed R42: 27k, Resistor_SMD:R_1206_3216Metric
- removed R43: 200, Resistor_SMD:R_1206_3216Metric
- removed R45: 3.3k, Resistor_SMD:R_1206_3216Metric
- added FB1: FerriteBead, Inductor_SMD:L_1206_3216Metric, F.Cu at (132.0, 59.2)
- added U3: ~, Dam_libkicad:PAD_Connector, F.Cu at (35.6, 75.6)
- added U4: ~, Dam_libkicad:PAD_Connector, F.Cu at (35.5, 62.2)
- C1, C2: footprint Dam_libkicad:1206 -> Dam_libkicad:0603
- C23: footprint Capacitor_SMD:C_0201_0603Metric -> Dam_libkicad:0603; moved to B.Cu
- C24, C25, C26, C27, C28, C3, C4, C5, C6, C7, C9: footprint Capacitor_SMD:C_1206_3216Metric -> Dam_libkicad:0603
- C44, C45, C46, C47: footprint Capacitor_SMD:C_1206_3216Metric_Pad1.33x1.80mm_HandSolder -> Dam_libkicad:0603
- IC1: footprint Dam_libkicad:SOP50P810X120-57N -> Dam_libkicad:QFN50P700X700X100-49N-D; moved to B.Cu
- Q2, Q3, Q4: footprint Package_TO_SOT_SMD:SOT-23 -> Package_TO_SOT_SMD:TO-263-2
- Q5, Q6, Q7: footprint Package_TO_SOT_SMD:SOT-23 -> Package_TO_SOT_SMD:TO-263-2; moved to B.Cu
- R1, R2, R25, R26, R27, R28, R29, R3, R30, R31, R32, R33, R34, R4, R5, R6, R7, R8: footprint Resistor_SMD:R_1206_3216Metric -> Dam_libkicad:0603
- R24: footprint Resistor_SMD:R_1206_3216Metric -> Dam_libkicad:0603; moved to B.Cu
- R35: value R -> 1; footprint Resistor_SMD:R_1206_3216Metric -> Dam_libkicad:0603; moved to B.Cu
- R46, R47, R48: footprint Resistor_SMD:R_1206_3216Metric_Pad1.30x1.75mm_HandSolder -> Dam_libkicad:0603
- R9: value 10k -> R; footprint Dam_libkicad:1206 -> Dam_libkicad:0603
- U5, U6, U7: value LMV321 -> ~; footprint Package_SO:SOIC-8_3.9x4.9mm_P1.27mm -> Dam_libkicad:PAD_Connector
- moved U5 165.0 mm to (35.3, 48.5), turned to 180 degrees
- moved R35 142.2 mm to (71.1, 75.7)
- moved U6 106.8 mm to (101.0, 47.4), turned to -90 degrees
- moved Q2 106.6 mm to (44.7, 50.5), turned to 180 degrees
- moved Q4 105.8 mm to (44.9, 77.7), turned to 180 degrees
- moved Q3 105.8 mm to (44.9, 64.2), turned to 180 degrees
- moved Q5 105.5 mm to (48.5, 50.5)
- moved Q6 103.4 mm to (48.6, 64.2)
- moved Q7 102.2 mm to (48.6, 77.7)
- moved C23 99.9 mm to (71.1, 74.5), turned to 180 degrees
- moved R30 96.6 mm to (127.3, 39.0)
- moved U7 96.1 mm to (100.9, 83.1), turned to -90 degrees
- moved R24 95.9 mm to (71.2, 73.4), turned to 180 degrees
- moved R29 95.9 mm to (127.3, 36.9)
- moved R34 95.9 mm to (127.3, 47.7)
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Connections:
- C1 pad 2: R_SHUNT1_N -> GND
- C2 pad 2: R_SHUNT1_N -> GND
- C24 pad 1: Net-(IC1-DVDD) -> Net-(IC1-VREF)
- C24 pad 2: R_SHUNT1_N -> GND
- C25 pad 1: Net-(IC1-REF) -> Net-(C25-Pad1)
- C25 pad 2: R_SHUNT1_N -> GND
- C26 pad 2: R_SHUNT1_N -> GND
- C27 pad 2: R_SHUNT1_N -> GND
- C28 pad 2: R_SHUNT1_N -> GND
- C3 pad 1: Net-(IC1-BIAS) -> V_BAT
- C3 pad 2: R_SHUNT1_N -> GND
- C4 pad 1: Net-(IC1-BST_A) -> V_BAT
- C4 pad 2: MOTOR_U -> GND
- C44 pad 1: R_SHUNT1_N -> GND
- C44 pad 2: Net-(U2-3V3OUT) -> D+
- C45 pad 2: R_SHUNT1_N -> GND
- C46 pad 2: R_SHUNT1_N -> GND
- C5 pad 1: Net-(IC1-CP1) -> unconnected-(C5-Pad1)
- C5 pad 2: Net-(IC1-CP2) -> unconnected-(C5-Pad2)
- C6 pad 1: Net-(IC1-GVDD) -> unconnected-(C6-Pad1)
- C6 pad 2: R_SHUNT1_N -> GND
- C7 pad 1: Net-(IC1-BST_B) -> V_BAT
- C7 pad 2: MOTOR_U -> GND
- C9 pad 1: Net-(IC1-AVDD) -> unconnected-(C9-Pad1)
- C9 pad 2: R_SHUNT1_N -> GND
- D5 pad 1: R_SHUNT1_N -> GND
- IC1 pad 10: Net-(IC1-GAIN) -> GL_A
- IC1 pad 11: Net-(IC1-OC_ADJ) -> R_SHUNT1_P
- IC1 pad 12: DC_CAL -> R_SHUNT1_N
- IC1 pad 13: Net-(IC1-GVDD) -> R_SHUNT2_N
- IC1 pad 14: Net-(IC1-CP1) -> R_SHUNT1_P
- IC1 pad 15: Net-(IC1-CP2) -> GL_B
- IC1 pad 16: GDR_EN -> MOTOR_V
- IC1 pad 17: PWM_A_H -> GH_B
- IC1 pad 18: PWM_A_L -> GH_C
- IC1 pad 19: PWM_B_H -> MOTOR_W
- IC1 pad 20: PWM_B_L -> GL_C
- IC1 pad 21: PWM_C_H -> R_SHUNT1_P
- IC1 pad 22: PWM_C_L -> unconnected-(IC1-SNC-Pad22)
- IC1 pad 23: Net-(IC1-DVDD) -> SO_C
- IC1 pad 24: Net-(IC1-REF) -> SO_B
- IC1 pad 25: SO1 -> SO_A
- IC1 pad 26: SO2 -> Net-(IC1-VREF)
- IC1 pad 27: Net-(IC1-AVDD) -> unconnected-(IC1-DGND-Pad27)
- IC1 pad 28: R_SHUNT1_N -> unconnected-(IC1-NFAULT-Pad28)
- IC1 pad 29: V_BAT -> unconnected-(IC1-SDO-Pad29)
- IC1 pad 30: R_SHUNT1_N -> unconnected-(IC1-SDI-Pad30)
- IC1 pad 31: R_SHUNT2_P -> unconnected-(IC1-SCLK-Pad31)
- IC1 pad 32: R_SHUNT1_N -> unconnected-(IC1-NSCS-Pad32)
- IC1 pad 33: R_SHUNT1_P -> unconnected-(IC1-ENABLE-Pad33)
- IC1 pad 34: R_SHUNT1_N -> unconnected-(IC1-CAL-Pad34)
- IC1 pad 35: GL_C -> unconnected-(IC1-AGND-Pad35)
- IC1 pad 36: MOTOR_U -> unconnected-(IC1-DVDD-Pad36)
- IC1 pad 37: GH_C -> PWM_A_H
- IC1 pad 38: Net-(IC1-BST_C) -> PWM_A_L
- IC1 pad 39: R_SHUNT2_P -> PWM_B_H
- IC1 pad 40: GL_B -> PWM_B_L
- IC1 pad 41: MOTOR_U -> PWM_C_H
- IC1 pad 42: GH_B -> PWM_C_L
- IC1 pad 43: Net-(IC1-BST_B) -> unconnected-(IC1-BGND-Pad43)
- IC1 pad 44: R_SHUNT1_P -> unconnected-(IC1-CB-Pad44)
- IC1 pad 45: GL_A -> unconnected-(IC1-SW-Pad45)
- IC1 pad 46: MOTOR_U -> unconnected-(IC1-NC-Pad46)
- IC1 pad 47: GH_A -> unconnected-(IC1-VIN-Pad47)
- IC1 pad 48: Net-(IC1-BST_A) -> unconnected-(IC1-NSHDN-Pad48)
- IC1 pad 49: Net-(IC1-BIAS) -> unconnected-(IC1-THERMAL_PAD-Pad49)
- IC1 pad 5: nOCTW -> unconnected-(IC1-VCP-Pad5)
- IC1 pad 6: nFAULT -> unconnected-(IC1-VM-Pad6)
- IC1 pad 7: Net-(IC1-DTC) -> unconnected-(IC1-VDRAIN-Pad7)
- IC1 pad 8: Net-(IC1-M_PWM) -> GH_A
- IC1 pad 9: Net-(IC1-M_OC) -> MOTOR_U
- J6 pad A1: R_SHUNT1_N -> GND
- J6 pad A12: R_SHUNT1_N -> GND
- J6 pad A7: D- -> D+
- J6 pad B1: R_SHUNT1_N -> GND
- J6 pad B12: R_SHUNT1_N -> GND
- J6 pad B7: D- -> D+
- J6 pad S1: R_SHUNT1_N -> GND
- Q2 pad 1: V_BAT -> GH_C
- Q2 pad 2: Net-(Q2-G) -> MOTOR_W
- Q2 pad 3: MOTOR_U -> V_BAT
- Q3 pad 1: V_BAT -> GH_B
- Q3 pad 2: Net-(Q3-G) -> MOTOR_V
- Q3 pad 3: MOTOR_U -> V_BAT
- Q4 pad 1: V_BAT -> GH_A
- Q4 pad 2: Net-(Q4-G) -> MOTOR_U
- Q4 pad 3: MOTOR_U -> V_BAT
- Q5 pad 1: MOTOR_U -> GL_C
- Q5 pad 2: Net-(Q5-G) -> R_SHUNT1_P
- Q5 pad 3: R_SHUNT1_N -> MOTOR_W
- Q6 pad 1: MOTOR_U -> GL_B
- Q6 pad 2: Net-(Q6-G) -> R_SHUNT1_P
- Q6 pad 3: R_SHUNT2_P -> MOTOR_V
- Q7 pad 1: MOTOR_U -> GL_A
- Q7 pad 2: Net-(Q7-G) -> R_SHUNT1_P
- Q7 pad 3: R_SHUNT1_P -> MOTOR_U
- R27 pad 1: VIRTUAL_N -> PHV_U
- R27 pad 2: PHV_U -> MOTOR_U
- R28 pad 1: PHV_U -> VIRTUAL_N
- R28 pad 2: MOTOR_U -> PHV_V
- R29 pad 1: VIRTUAL_N -> PHV_V
- R29 pad 2: PHV_V -> MOTOR_V
- R3 pad 1: R_SHUNT1_N -> GND
- R3 pad 2: Net-(IC1-DTC) -> unconnected-(R3-Pad2)
- R30 pad 1: PHV_V -> VIRTUAL_N
- R30 pad 2: MOTOR_V -> PHV_W
- R31 pad 1: VIRTUAL_N -> PHV_W
- R31 pad 2: PHV_W -> MOTOR_W
- R32 pad 1: PHV_W -> GND
- R32 pad 2: MOTOR_W -> PHV_U
- R33 pad 1: R_SHUNT1_N -> GND
- R33 pad 2: PHV_U -> PHV_V
- R34 pad 1: R_SHUNT1_N -> GND
- R34 pad 2: PHV_V -> PHV_W
- R35 pad 2: PHV_W -> GND
- R4 pad 1: R_SHUNT1_N -> GND
- R4 pad 2: Net-(IC1-M_PWM) -> unconnected-(R4-Pad2)
- R5 pad 1: R_SHUNT1_N -> GND
- R5 pad 2: Net-(IC1-M_OC) -> unconnected-(R5-Pad2)
- R6 pad 1: Net-(IC1-OC_ADJ) -> Net-(R6-Pad1)
- R7 pad 2: Net-(IC1-GAIN) -> unconnected-(R7-Pad2)
- R8 pad 1: R_SHUNT1_N -> GND
- R8 pad 2: Net-(IC1-OC_ADJ) -> Net-(R6-Pad1)
- R9 pad 1: +5V -> VIRTUAL_N
- R9 pad 2: RST -> PHV_U
- U1 pad 1: PWM_A_H -> PWM_B_L
- U1 pad 10: PWM_C_H -> VIRTUAL_N
- U1 pad 13: PWM_B_L -> PWM_A_H
- U1 pad 15: PWM_A_L -> PWM_C_H
- U1 pad 2: unconnected-(U1-(4/T0)PD4-Pad2) -> PWM_A_L
- U1 pad 21: R_SHUNT1_N -> GND
- U1 pad 23: unconnected-(U1-(A0)PC0-Pad23) -> PHV_W
- U1 pad 24: unconnected-(U1-(A1)PC1-Pad24) -> PHV_V
- U1 pad 25: unconnected-(U1-(A2)PC2-Pad25) -> PHV_U
- U1 pad 3: R_SHUNT1_N -> GND
- U1 pad 32: unconnected-(U1-(2/INT0)PD2-Pad32) -> PWM_C_L
- U1 pad 5: R_SHUNT1_N -> GND
- U1 pad 9: PWM_C_L -> unconnected-(U1-(5/OC0B/T1)PD5-Pad9)
- U2 pad 10: Net-(U2-3V3OUT) -> D+
- U2 pad 11: Net-(U2-3V3OUT) -> D+
- U2 pad 13: R_SHUNT1_N -> GND
- U2 pad 3: Net-(U2-3V3OUT) -> D+
- U2 pad 5: R_SHUNT1_N -> GND
- U2 pad 9: D- -> D+
- U5 pad 1: PHV_U -> MOTOR_W
- U6 pad 1: PHV_V -> V_BAT
- U7 pad 1: PHV_W -> GND
- Y1 pad 2: R_SHUNT1_N -> GND
Routing:
- net V_BAT: track 0.00 -> 95.1 mm
- net MOTOR_U: track 0.00 -> 68.0 mm
- net R_SHUNT1_P: track 0.00 -> 61.2 mm, vias 0 -> 5
- net MOTOR_W: track 0.00 -> 55.6 mm
- net GL_A: track 0.00 -> 46.2 mm
- net GH_A: track 0.00 -> 40.1 mm, vias 0 -> 1
- net MOTOR_V: track 0.00 -> 36.9 mm, vias 0 -> 1
- net GL_C: track 0.00 -> 34.4 mm
- net GL_B: track 0.00 -> 34.1 mm
- net GH_C: track 0.00 -> 24.8 mm, vias 0 -> 1
- net PWM_A_H: track 0.00 -> 19.0 mm, vias 0 -> 1
- net PWM_B_H: track 0.00 -> 18.2 mm, vias 0 -> 1
- net PWM_C_H: track 0.00 -> 17.5 mm, vias 0 -> 1
- net GH_B: track 0.00 -> 17.4 mm, vias 0 -> 1
- net R_SHUNT1_N: track 0.00 -> 6.50 mm, vias 0 -> 1
Other:
- board outline added: 72.7 x 41.5 mm

Commit message: v2 80%
Parts:
- removed C23: C, Dam_libkicad:0603
- removed C25, C44: 1uF, Dam_libkicad:0603
- removed C45: 4.7uF_16V, Dam_libkicad:0603
- removed C46, C47: 100nF, Dam_libkicad:0603
- removed D5: LED, LED_SMD:LED_1206_3216Metric_Pad1.42x1.75mm_HandSolder
- removed D7: RX, LED_SMD:LED_1206_3216Metric_Pad1.42x1.75mm_HandSolder
- removed D8: TX, LED_SMD:LED_1206_3216Metric_Pad1.42x1.75mm_HandSolder
- removed F1: Fuse, Fuse:Fuse_1206_3216Metric_Pad1.42x1.75mm_HandSolder
- removed FB1: FerriteBead, Inductor_SMD:L_1206_3216Metric
- removed J6: USB_C_Receptacle_USB2.0, Connector_USB:USB_C_Receptacle_GCT_USB4105-xx-A_16P_TopMnt_Horizontal
- removed R35: 1, Dam_libkicad:0603
- removed R46, R47, R48: 1K, Dam_libkicad:0603
- removed U2: FT230XS, Package_SO:SSOP-16_5.3x6.2mm_P0.65mm
- removed U3, U4, U5, U6, U7: ~, Dam_libkicad:PAD_Connector
- added C10: >10uF, Dam_libkicad:1206, F.Cu at (72.7, 72.8)
- added C11: 1uF, Dam_libkicad:1206, B.Cu at (83.3, 73.0)
- added C12: 1uF, Dam_libkicad:1206, F.Cu at (99.5, 78.4)
- added C13: C_Polarized, Capacitor_THT:CP_Radial_D18.0mm_P7.50mm, F.Cu at (103.6, 61.5)
- added C8: 1uF, Dam_libkicad:1206, F.Cu at (72.7, 70.7)
- added D1: D_Schottky_Filled, Dam_libkicad:1206, F.Cu at (83.4, 77.2)
- added H1: Cosses PCB 90°, Dam_libkicad:12177561, F.Cu at (99.8, 43.6)
- added H2: Cosses PCB 90°, Dam_libkicad:12177561, F.Cu at (99.8, 84.2)
- added H3: Cosses PCB 90°, Dam_libkicad:12177561, F.Cu at (37.0, 75.5)
- added H4: Cosses PCB 90°, Dam_libkicad:12177561, F.Cu at (36.9, 59.9)
- added H5: Cosses PCB 90°, Dam_libkicad:12177561, F.Cu at (36.9, 44.5)
- added J1: Conn_01x03, Connector_PinSocket_2.54mm:PinSocket_1x03_P2.54mm_Horizontal, B.Cu at (124.3, 49.0)
- added J2: Prog, Connector_PinHeader_2.54mm:PinHeader_1x04_P2.54mm_Vertical, F.Cu at (82.8, 47.8)
- added L1: L, Inductor_SMD:L_Ferrocore_DLG-1005, F.Cu at (90.6, 77.2)
- added R10: R, Dam_libkicad:0603, B.Cu at (74.4, 55.3)
- added R11: R, Dam_libkicad:0603, B.Cu at (74.4, 56.7)
- added R12: R, Dam_libkicad:0603, B.Cu at (74.4, 58.0)
- added R13: R, Dam_libkicad:0603, B.Cu at (74.4, 59.4)
- added R14: 10k, Dam_libkicad:0603, B.Cu at (74.4, 51.3)
- added R15: 100k, Dam_libkicad:1206, F.Cu at (76.3, 73.4)
- added R16: 10k, Dam_libkicad:1206, F.Cu at (93.2, 51.9)
- C1, C2, C26, C27, C28, C3, C4, C7, R1, R2, R27, R28, R29, R30, R31, R32, R33, R34, R9: footprint Dam_libkicad:0603 -> Dam_libkicad:1206
- C24: footprint Dam_libkicad:0603 -> Dam_libkicad:1206; moved to B.Cu
- C5: value 22nF -> 47nF; footprint Dam_libkicad:0603 -> Dam_libkicad:1206
- C6: value 2.2nF -> 1uF; moved to B.Cu
- C9: value 1uF -> 10uF; footprint Dam_libkicad:0603 -> Dam_libkicad:1206
- IC1: value DRV8302DCA -> DRV8323RHRGZT; footprint Dam_libkicad:QFN50P700X700X100-49N-D -> Dam_libkicad:DRV8323RHRGZT
- Q2, Q3, Q4, Q5, Q6, Q7: footprint Package_TO_SOT_SMD:TO-263-2 -> Dam_libkicad:D2PAK
- R24: footprint Dam_libkicad:0603 -> Resistor_SMD:R_Shunt_Vishay_WSR2_WSR3
- R3, R4: footprint Dam_libkicad:0603 -> Resistor_SMD:R_Shunt_Vishay_WSR2_WSR3; moved to B.Cu
- R5, R6, R7, R8: moved to B.Cu
- moved R29 67.9 mm to (65.3, 64.5), turned to -90 degrees
- moved R31 65.1 mm to (63.8, 55.1), turned to -90 degrees
- moved R3 63.9 mm to (58.8, 69.8), turned to -90 degrees
- moved R34 61.7 mm to (65.8, 52.3), turned to -90 degrees
- moved C7 61.6 mm to (61.2, 74.0)
- moved R33 59.8 mm to (67.9, 52.3), turned to -90 degrees
- moved R4 59.1 mm to (61.7, 45.2)
- moved Y1 58.5 mm to (78.8, 61.0), turned to 90 degrees
- moved R32 58.0 mm to (70.0, 52.3), turned to -90 degrees
- moved C3 57.4 mm to (60.5, 59.3)
- moved R27 56.3 mm to (68.8, 64.5), turned to -90 degrees
- moved C5 55.7 mm to (75.5, 79.0)
- moved R30 55.4 mm to (73.3, 51.4), turned to 180 degrees
- moved R7 53.1 mm to (74.4, 60.7), turned to 180 degrees
- moved C4 52.9 mm to (61.2, 47.9)
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Connections:
- C24 pad 1: Net-(IC1-VREF) -> DVDD
- C5 pad 1: unconnected-(C5-Pad1) -> Net-(IC1-CPH)
- C5 pad 2: unconnected-(C5-Pad2) -> Net-(IC1-CPL)
- C6 pad 1: unconnected-(C6-Pad1) -> AGND
- C6 pad 2: GND -> DVDD
- C9 pad 1: unconnected-(C9-Pad1) -> V_BAT
- IC1 pad 1: unconnected-(IC1-FB-Pad1) -> FB
- IC1 pad 12: R_SHUNT1_N -> GND
- IC1 pad 13: R_SHUNT2_N -> GND
- IC1 pad 14: R_SHUNT1_P -> R_SHUNT2_P
- IC1 pad 2: unconnected-(IC1-PGND-Pad2) -> GND
- IC1 pad 21: R_SHUNT1_P -> R_SHUNT3_P
- IC1 pad 22: unconnected-(IC1-SNC-Pad22) -> GND
- IC1 pad 26: Net-(IC1-VREF) -> DVDD
- IC1 pad 27: unconnected-(IC1-DGND-Pad27) -> GND
- IC1 pad 28: unconnected-(IC1-NFAULT-Pad28) -> nFAULT
- IC1 pad 29: unconnected-(IC1-SDO-Pad29) -> MODE
- IC1 pad 3: unconnected-(IC1-CPL-Pad3) -> Net-(IC1-CPL)
- IC1 pad 30: unconnected-(IC1-SDI-Pad30) -> IDRIVE
- IC1 pad 31: unconnected-(IC1-SCLK-Pad31) -> VDS
- IC1 pad 32: unconnected-(IC1-NSCS-Pad32) -> GAIN
- IC1 pad 33: unconnected-(IC1-ENABLE-Pad33) -> ENABLE
- IC1 pad 34: unconnected-(IC1-CAL-Pad34) -> CAL
- IC1 pad 35: unconnected-(IC1-AGND-Pad35) -> AGND
- IC1 pad 36: unconnected-(IC1-DVDD-Pad36) -> DVDD
- IC1 pad 4: unconnected-(IC1-CPH-Pad4) -> Net-(IC1-CPH)
- IC1 pad 43: unconnected-(IC1-BGND-Pad43) -> GND
- IC1 pad 44: unconnected-(IC1-CB-Pad44) -> CB
- IC1 pad 45: unconnected-(IC1-SW-Pad45) -> SW
- IC1 pad 47: unconnected-(IC1-VIN-Pad47) -> V_BAT
- IC1 pad 48: unconnected-(IC1-NSHDN-Pad48) -> Net-(IC1-NSHDN)
- IC1 pad 49: unconnected-(IC1-THERMAL_PAD-Pad49) -> GND
- IC1 pad 5: unconnected-(IC1-VCP-Pad5) -> V_BAT
- IC1 pad 6: unconnected-(IC1-VM-Pad6) -> Net-(IC1-VM)
- IC1 pad 7: unconnected-(IC1-VDRAIN-Pad7) -> V_BAT
- Q5 pad 2: R_SHUNT1_P -> R_SHUNT3_P
- Q6 pad 2: R_SHUNT1_P -> R_SHUNT2_P
- R1 pad 1: nOCTW -> +5V
- R1 pad 2: VDD_3V3 -> FB
- R2 pad 1: nFAULT -> FB
- R2 pad 2: VDD_3V3 -> GND
- R24 pad 2: R_SHUNT1_N -> GND
- R3 pad 1: GND -> R_SHUNT2_P
- R3 pad 2: unconnected-(R3-Pad2) -> GND
- R4 pad 1: GND -> R_SHUNT3_P
- R4 pad 2: unconnected-(R4-Pad2) -> GND
- R5 pad 1: GND -> DVDD
- R5 pad 2: unconnected-(R5-Pad2) -> MODE
- R6 pad 1: Net-(R6-Pad1) -> MODE
- R6 pad 2: VDD_3V3 -> AGND
- R7 pad 1: VDD_3V3 -> DVDD
- R7 pad 2: unconnected-(R7-Pad2) -> GAIN
- R8 pad 1: GND -> GAIN
- R8 pad 2: Net-(R6-Pad1) -> AGND
- U1 pad 1: PWM_B_L -> unconnected-(U1-(3/OC2B/INT1)PD3-Pad1)
- U1 pad 12: unconnected-(U1-(8)PB0-Pad12) -> PWM_A_L
- U1 pad 16: unconnected-(U1-(12/MISO)PB4-Pad16) -> PWM_B_L
- U1 pad 17: unconnected-(U1-(13/SCK)PB5-Pad17) -> PWM_C_L
- U1 pad 2: PWM_A_L -> unconnected-(U1-(4/T0)PD4-Pad2)
- U1 pad 32: PWM_C_L -> unconnected-(U1-(2/INT0)PD2-Pad32)
Routing:
- net GND: track 0.00 -> 335.7 mm, vias 0 -> 5
- net V_BAT: track 95.1 -> 161.5 mm, vias 0 -> 2
- net +5V: track 0.00 -> 56.0 mm
- net PHV_U: track 0.00 -> 49.1 mm, vias 0 -> 2
- net PHV_V: track 0.00 -> 46.7 mm, vias 0 -> 2
- net R_SHUNT3_P: track 0.00 -> 40.0 mm
- net PHV_W: track 0.00 -> 37.5 mm, vias 0 -> 2
- net FB: track 0.00 -> 32.6 mm, vias 0 -> 1
- net R_SHUNT1_P: track 61.2 -> 29.1 mm, vias 5 -> 0
- net DVDD: track 0.00 -> 31.3 mm
- net R_SHUNT2_P: track 0.00 -> 26.6 mm, vias 0 -> 2
- net CB: track 0.00 -> 24.4 mm, vias 0 -> 1
- net PWM_C_L: track 0.00 -> 23.6 mm, vias 0 -> 1
- net MOTOR_V: track 36.9 -> 60.2 mm, vias 1 -> 2
- net VIRTUAL_N: track 0.00 -> 21.8 mm
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- added copper zone on B.Cu, net GND
- added copper zone on F.Cu, net GND
Other:
- board size 72.7 x 41.5 mm -> 76.3 x 44.9 mm
